File: hardware/0.2/n64.sch (KiCad schematic (older format))
At the start: 46 parts, among them J1 , J2 Conn_01x05_Male, J3 Conn_01x03_Male, J4 Conn_02x08_Counter_Clockwise, J5 Conn_01x09_Male, U1 ICE40HX4K-TQ144, U2 ATtiny45-20PU, U3 S25FL064, U4 TLV73312PDBV, U5 IS42S16320D, U6 Multicomp_Oscillator, U7 Nintendo_64_Logo, U8 ATtiny45V-10PU

Commit message: some changes
Parts:
- removed D2: LED, LED_SMD:LED_0603_1608Metric_Pad1.05x0.95mm_HandSolder, symbol Device:LED
- removed R6: 1k, Resistor_SMD:R_0603_1608Metric_Pad1.05x0.95mm_HandSolder, symbol Device:R_Small
- removed TP2: TestPoint, TestPoint:TestPoint_Pad_D1.5mm, symbol Connector:TestPoint
- J2: value Conn_01x05_Male -> Conn_01x07_Male; footprint Connector_PinHeader_2.54mm:PinHeader_1x05_P2.54mm_Vertical -> Connector_PinHeader_2.54mm:PinHeader_1x07_P2.54mm_Vertical; symbol Connector:Conn_01x05_Male -> Connector:Conn_01x07_Male
Connections:
- net FLASH_DI: now also U1.67 (IOB_105_SDO); no longer U1.68 (IOB_106_SDI)
- net FLASH_DO: now also U1.68 (IOB_106_SDI); no longer U1.67 (IOB_105_SDO)
- net GND: now also J2.7 (Pin_7); no longer J2.5 (Pin_5)
- net at U5.36 (NC): now also U1.107 (IOR_167)
- net CDONE: now reaches U1.65 (CDONE)
- net CDONE: now also J2.6 (Pin_6)
- net !CRESET: now reaches R4.1, U1.66 (~CRESET)
- net !CRESET: now also J2.5 (Pin_5)
- removed net A12: U1.107 (IOR_167), U5.36 (NC)
Other:
- moved on the sheet: 1v2, 2v5, 3v3, C1, C10, C2, C3, C4, C5, C6, C7, C8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
